Commit message: Updata dex-retargeting lib to 0.4.6

File: assets/inspire_hand_org/inspire_hand_left.urdf (robot description, URDF)
Before this commit: robot h1, 18 links, 17 joints
Joints:
- joint L_thumb_proximal_pitch_joint: limit lower=0.0 upper=0.67 effort=1 velocity=0.5 -> lower=0.0 upper=0.5 effort=1 velocity=0.5
- joint L_thumb_proximal_yaw_joint: limit lower=0.0 upper=1.69 effort=1 velocity=0.5 -> lower=-0.1 upper=1.3 effort=1 velocity=0.5

File: assets/inspire_hand_org/inspire_hand_right.urdf (robot description, URDF)
Before this commit: robot h1, 18 links, 17 joints
Joints:
- joint R_thumb_proximal_yaw_joint: limit lower=-0.1 upper=1.8 effort=1 velocity=0.5 -> lower=-0.1 upper=1.3 effort=1 velocity=0.5
