Commit message: Change parameter of Inspire Hand URDF to match the  real environment

File: assets/inspire_hand/inspire_hand_left.urdf (robot description, URDF)
Before this commit: robot h1, 18 links, 17 joints
Joints:
- joint L_index_intermediate_joint: mimic joint=L_index_proximal_joint multiplier=1 offset=0 -> joint=L_index_proximal_joint multiplier=1.117 offset=-0.187
- joint L_index_proximal_joint: limit lower=0 upper=1.7 effort=1 velocity=0.5 -> lower=0 upper=1.3090 effort=1 velocity=0.5
- joint L_middle_intermediate_joint: mimic joint=L_middle_proximal_joint multiplier=1 offset=0 -> joint=L_middle_proximal_joint multiplier=1.117 offset=-0.187
- joint L_middle_proximal_joint: limit lower=0 upper=1.7 effort=1 velocity=0.5 -> lower=0 upper=1.3090 effort=1 velocity=0.5
- joint L_pinky_intermediate_joint: mimic joint=L_pinky_proximal_joint multiplier=1 offset=0 -> joint=L_pinky_proximal_joint multiplier=1.117 offset=-0.187
- joint L_pinky_proximal_joint: limit lower=0 upper=1.7 effort=1 velocity=0.5 -> lower=0 upper=1.3090 effort=1 velocity=0.5
- joint L_ring_intermediate_joint: mimic joint=L_ring_proximal_joint multiplier=1 offset=0 -> joint=L_ring_proximal_joint multiplier=1.117 offset=-0.187
- joint L_ring_proximal_joint: limit lower=0 upper=1.7 effort=1 velocity=0.5 -> lower=0 upper=1.3090 effort=1 velocity=0.5
- joint L_thumb_distal_joint: mimic joint=L_thumb_proximal_pitch_joint multiplier=2.4 offset=0 -> joint=L_thumb_proximal_pitch_joint multiplier=0.864 offset=0.907
- joint L_thumb_intermediate_joint: mimic joint=L_thumb_proximal_pitch_joint multiplier=1.6 offset=0 -> joint=L_thumb_proximal_pitch_joint multiplier=1.142 offset=0.490
- joint L_thumb_proximal_pitch_joint: limit lower=0.0 upper=0.67 effort=1 velocity=0.5 -> lower=0.0 upper=0.4712 effort=1 velocity=0.5
- joint L_thumb_proximal_yaw_joint: limit lower=0.0 upper=1.69 effort=1 velocity=0.5 -> lower=0.0 upper=1.3090 effort=1 velocity=0.5

File: assets/inspire_hand/inspire_hand_right.urdf (robot description, URDF)
Before this commit: robot h1, 18 links, 17 joints
Joints:
- joint R_index_proximal_joint: limit lower=0 upper=1.7 effort=1 velocity=0.5 -> lower=0 upper=1.3090 effort=1 velocity=0.5
- joint R_middle_intermediate_joint: mimic joint=R_middle_proximal_joint multiplier=1 offset=0 -> joint=R_middle_proximal_joint multiplier=1.117 offset=-0.187
- joint R_middle_proximal_joint: limit lower=0 upper=1.7 effort=1 velocity=0.5 -> lower=0 upper=1.3090 effort=1 velocity=0.5
- joint R_pinky_intermediate_joint: mimic joint=R_pinky_proximal_joint multiplier=1 offset=0 -> joint=R_pinky_proximal_joint multiplier=1.117 offset=-0.187
- joint R_pinky_proximal_joint: limit lower=0 upper=1.7 effort=1 velocity=0.5 -> lower=0 upper=1.3090 effort=1 velocity=0.5
- joint R_ring_intermediate_joint: mimic joint=R_ring_proximal_joint multiplier=1 offset=0 -> joint=R_ring_proximal_joint multiplier=1.117 offset=-0.187
- joint R_ring_proximal_joint: limit lower=0 upper=1.7 effort=1 velocity=0.5 -> lower=0 upper=1.3090 effort=1 velocity=0.5
- joint R_thumb_distal_joint: mimic joint=R_thumb_proximal_pitch_joint multiplier=2.4 offset=0 -> joint=R_thumb_proximal_pitch_joint multiplier=0.864 offset=0.907
- joint R_thumb_intermediate_joint: mimic joint=R_thumb_proximal_pitch_joint multiplier=1.6 offset=0 -> joint=R_thumb_proximal_pitch_joint multiplier=1.142 offset=0.490
- joint R_thumb_proximal_pitch_joint: limit lower=0.0 upper=0.5 effort=1 velocity=0.5 -> lower=0.0 upper=0.4712 effort=1 velocity=0.5
- joint R_thumb_proximal_yaw_joint: limit lower=-0.1 upper=1.8 effort=1 velocity=0.5 -> lower=0 upper=1.3090 effort=1 velocity=0.5
