Commit message: Change the file path of URDF imported into pinocchio. Now it doesn't require path changing in franka urdf file

File: assets/franka_gym/robots/franka_panda.urdf (robot description, URDF)
Before this commit: robot panda, 8 links, 7 joints
Links:
- link panda_link0: geometry collision mesh filename=package://franka_description/meshes/collision/link0.stl; visual mesh filename=package://franka_description/meshes/visual/link0.dae
- link panda_link1: geometry collision mesh filename=package://franka_description/meshes/collision/link1.stl; visual mesh filename=package://franka_description/meshes/visual/link1.dae
- link panda_link2: geometry collision mesh filename=package://franka_description/meshes/collision/link2.stl; visual mesh filename=package://franka_description/meshes/visual/link2.dae
- link panda_link3: geometry collision mesh filename=package://franka_description/meshes/collision/link3.stl; visual mesh filename=package://franka_description/meshes/visual/link3.dae
- link panda_link4: geometry collision mesh filename=package://franka_description/meshes/collision/link4.stl; visual mesh filename=package://franka_description/meshes/visual/link4.dae
- link panda_link5: geometry collision mesh filename=package://franka_description/meshes/collision/link5.stl; visual mesh filename=package://franka_description/meshes/visual/link5.dae
- link panda_link6: geometry collision mesh filename=package://franka_description/meshes/collision/link6.stl; visual mesh filename=package://franka_description/meshes/visual/link6.dae
- link panda_link7: geometry collision mesh filename=package://franka_description/meshes/collision/link7.stl; visual mesh filename=package://franka_description/meshes/visual/link7.dae

Commit message: connect inspire hand and franka urdf

File: assets/franka_gym/robots/franka_panda.urdf (robot description, URDF)
Before this commit: robot panda, 8 links, 7 joints
Links:
- link panda_link0: geometry collision mesh filename=package://franka_description/meshes/collision/link0.stl; visual mesh filename=../meshes/visual/link0.dae
- link panda_link1: geometry collision mesh filename=package://franka_description/meshes/collision/link1.stl; visual mesh filename=../meshes/visual/link1.dae
- link panda_link2: geometry collision mesh filename=package://franka_description/meshes/collision/link2.stl; visual mesh filename=../meshes/visual/link2.dae
- link panda_link3: geometry collision mesh filename=package://franka_description/meshes/collision/link3.stl; visual mesh filename=../meshes/visual/link3.dae
- link panda_link4: geometry collision mesh filename=package://franka_description/meshes/collision/link4.stl; visual mesh filename=../meshes/visual/link4.dae
- link panda_link5: geometry collision mesh filename=package://franka_description/meshes/collision/link5.stl; visual mesh filename=../meshes/visual/link5.dae
- link panda_link6: geometry collision mesh filename=package://franka_description/meshes/collision/link6.stl; visual mesh filename=../meshes/visual/link6.dae
- link panda_link7: geometry collision mesh filename=package://franka_description/meshes/collision/link7.stl; visual mesh filename=../meshes/visual/link7.dae

File: assets/franka_inspire_hand/franka_description/robots/franka_panda_right.urdf (robot description, URDF)
Before this commit: robot panda, 26 links, 25 joints
Links:
- removed link R_hand_base_link
- removed link R_index_intermediate
- removed link R_index_proximal
- removed link R_index_tip
- removed link R_middle_intermediate
- removed link R_middle_proximal
- removed link R_middle_tip
- removed link R_pinky_intermediate
- removed link R_pinky_proximal
- removed link R_pinky_tip
- removed link R_ring_intermediate
- removed link R_ring_proximal
- removed link R_ring_tip
- removed link R_thumb_distal
- removed link R_thumb_intermediate
- removed link R_thumb_proximal
- removed link R_thumb_proximal_base
- removed link R_thumb_tip
- added link hand_base_link, mass 0.14143; collision box size=0.0125 0.0111 0.0089; collision box size=0.0125 0.0111 0.0089
- added link index_intermediate, mass 0.0045683; collision mesh filename=meshes/collision/right_index_intermediate.obj; visual mesh filename=meshes/visual/right_index_intermediate.glb
- added link index_proximal, mass 0.0042403; collision mesh filename=meshes/collision/right_index_proximal.obj; visual mesh filename=meshes/visual/right_index_proximal.glb
- added link index_tip
- added link middle_intermediate, mass 0.0050396; collision mesh filename=meshes/collision/right_middle_intermediate.obj; visual mesh filename=meshes/visual/right_middle_intermediate.glb
- added link middle_proximal, mass 0.0042403; collision mesh filename=meshes/collision/right_index_proximal.obj; visual mesh filename=meshes/visual/right_index_proximal.glb
- added link middle_tip
- added link pinky_intermediate, mass 0.0035996; collision mesh filename=meshes/collision/right_pinky_intermediate.obj; visual mesh filename=meshes/visual/right_pinky_intermediate.glb
- added link pinky_proximal, mass 0.0042403; collision mesh filename=meshes/collision/right_index_proximal.obj; visual mesh filename=meshes/visual/right_index_proximal.glb
- added link pinky_tip
- added link ring_intermediate, mass 0.0045683; collision mesh filename=meshes/collision/right_index_intermediate.obj; visual mesh filename=meshes/visual/right_index_intermediate.glb
- added link ring_proximal, mass 0.0042403; collision mesh filename=meshes/collision/right_index_proximal.obj; visual mesh filename=meshes/visual/right_index_proximal.glb
- added link ring_tip
- added link thumb_distal, mass 0.0033441; collision mesh filename=meshes/collision/right_thumb_distal.obj; visual mesh filename=meshes/visual/right_thumb_distal.glb
- added link thumb_intermediate, mass 0.0037847; collision mesh filename=meshes/collision/right_thumb_intermediate.obj; visual mesh filename=meshes/visual/right_thumb_intermediate.glb
- added link thumb_proximal, mass 0.0066075; collision mesh filename=meshes/collision/right_thumb_proximal.obj; visual mesh filename=meshes/visual/right_thumb_proximal.glb
- added link thumb_proximal_base, mass 0.0018869; collision mesh filename=meshes/collision/right_thumb_proximal_base.obj; visual mesh filename=meshes/visual/right_thumb_proximal_base.glb
- added link thumb_tip
Joints:
- removed joint R_index_intermediate_joint
- removed joint R_index_proximal_joint
- removed joint R_index_tip_joint
- removed joint R_middle_intermediate_joint
- removed joint R_middle_proximal_joint
- removed joint R_middle_tip_joint
- removed joint R_pinky_intermediate_joint
- removed joint R_pinky_proximal_joint
- removed joint R_pinky_tip_joint
- removed joint R_ring_intermediate_joint
- removed joint R_ring_proximal_joint
- removed joint R_ring_tip_joint
- removed joint R_thumb_distal_joint
- removed joint R_thumb_intermediate_joint
- removed joint R_thumb_proximal_pitch_joint
- removed joint R_thumb_proximal_yaw_joint
- removed joint R_thumb_tip_joint
- added joint index_intermediate_joint: type revolute, parent index_proximal, child index_intermediate, origin xyz=-0.0026138 0.032026 -0.001 rpy=0 0 0, axis 0 0 1, limit lower=-0.04545 upper=1.56 effort=1 velocity=0.5, mimic joint=index_proximal_joint multiplier=1.06399 offset=-0.04545
- added joint index_proximal_joint: type revolute, parent hand_base_link, child index_proximal, origin xyz=0.00028533 -0.13653 -0.032268 rpy=-3.1067 0 0, axis 0 0 1, limit lower=0 upper=1.47 effort=1 velocity=0.5
- added joint index_tip_joint: type fixed, parent index_intermediate, child index_tip, origin xyz=-0.0008 0.045 -0.005 rpy=0 0 0
- added joint middle_intermediate_joint: type revolute, parent middle_proximal, child middle_intermediate, origin xyz=-0.0024229 0.032041 -0.001 rpy=0 0 0, axis 0 0 1, limit lower=-0.04545 upper=1.56 effort=1 velocity=0.5, mimic joint=middle_proximal_joint multiplier=1.06399 offset=-0.04545
- added joint middle_proximal_joint: type revolute, parent hand_base_link, child middle_proximal, origin xyz=0.00028533 -0.1371 -0.01295 rpy=-3.1416 0 0, axis 0 0 1, limit lower=0 upper=1.47 effort=1 velocity=0.5
- added joint middle_tip_joint: type fixed, parent middle_intermediate, child middle_tip, origin xyz=-0.001 0.048 -0.005 rpy=0 0 0
- added joint pinky_intermediate_joint: type revolute, parent pinky_proximal, child pinky_intermediate, origin xyz=-0.0024229 0.032041 -0.001 rpy=0 0 0, axis 0 0 1, limit lower=-0.04545 upper=1.56 effort=1 velocity=0.5, mimic joint=pinky_proximal_joint multiplier=1.06399 offset=-0.04545
- added joint pinky_proximal_joint: type revolute, parent hand_base_link, child pinky_proximal, origin xyz=0.00028533 -0.13571 0.025488 rpy=3.0369 0 0, axis 0 0 1, limit lower=0 upper=1.47 effort=1 velocity=0.5
- added joint pinky_tip_joint: type fixed, parent pinky_intermediate, child pinky_tip, origin xyz=-0.0008 0.037 -0.005 rpy=0 0 0
- added joint ring_intermediate_joint: type revolute, parent ring_proximal, child ring_intermediate, origin xyz=-0.0024229 0.032041 -0.001 rpy=0 0 0, axis 0 0 1, limit lower=-0.04545 upper=1.56 effort=1 velocity=0.5, mimic joint=ring_proximal_joint multiplier=1.06399 offset=-0.04545
- added joint ring_proximal_joint: type revolute, parent hand_base_link, child ring_proximal, origin xyz=0.00028533 -0.13691 0.0062872 rpy=3.0892 0 0, axis 0 0 1, limit lower=0 upper=1.47 effort=1 velocity=0.5
- added joint ring_tip_joint: type fixed, parent ring_intermediate, child ring_tip, origin xyz=-0.0008 0.045 -0.005 rpy=0 0 0
- added joint thumb_distal_joint: type revolute, parent thumb_intermediate, child thumb_distal, origin xyz=0.020248 0.010156 -0.0012 rpy=0 0 0, axis 0 0 1, limit lower=0 upper=0.4 effort=1 velocity=0.5, mimic joint=thumb_proximal_pitch_joint multiplier=0.667 offset=0
- added joint thumb_intermediate_joint: type revolute, parent thumb_proximal, child thumb_intermediate, origin xyz=0.04407 0.034553 -0.0008 rpy=0 0 0, axis 0 0 1, limit lower=0 upper=0.8 effort=1 velocity=0.5, mimic joint=thumb_proximal_pitch_joint multiplier=1.334 offset=0
- added joint thumb_proximal_pitch_joint: type revolute, parent thumb_proximal_base, child thumb_proximal, origin xyz=-0.0088099 0.010892 -0.00925 rpy=1.5708 0 2.8587, axis 0 0 1, limit lower=0 upper=0.6 effort=1 velocity=0.5
- added joint thumb_proximal_yaw_joint: type revolute, parent hand_base_link, child thumb_proximal_base, origin xyz=-0.01696 -0.0691 -0.02045 rpy=1.5708 -1.5708 0, axis 0 0 -1, limit lower=0.0 upper=1.308 effort=1 velocity=0.5
- added joint thumb_tip_joint: type fixed, parent thumb_distal, child thumb_tip, origin xyz=0.0202 0.0140 -0.006 rpy=0 0 0
- joint panda_hand_joint: child R_hand_base_link -> hand_base_link

File: assets/franka_pinocchio/robots/franka_panda.urdf (robot description, URDF)
Before this commit: robot panda, 8 links, 7 joints
Joints:
- joint panda_joint1: limit lower=-3 upper=3 effort=87 velocity=2.1750 -> lower=-2.8973 upper=2.8973 effort=87 velocity=2.1750
- joint panda_joint2: limit lower=-3 upper=3 effort=87 velocity=2.1750 -> lower=-1.7628 upper=1.7628 effort=87 velocity=2.1750
- joint panda_joint3: limit lower=-3 upper=3 effort=87 velocity=2.1750 -> lower=-2.8973 upper=2.8973 effort=87 velocity=2.1750
- joint panda_joint4: limit lower=-3 upper=3 effort=87 velocity=2.1750 -> lower=-3.0718 upper=-0.0698 effort=87 velocity=2.1750
- joint panda_joint5: limit lower=-3 upper=3 effort=87 velocity=2.1750 -> lower=-2.8973 upper=2.8973 effort=87 velocity=2.1750
- joint panda_joint6: limit lower=-3 upper=3 effort=87 velocity=2.1750 -> lower=-0.0175 upper=3.7525 effort=87 velocity=2.1750
- joint panda_joint7: limit lower=-3 upper=3 effort=87 velocity=2.1750 -> lower=-2.8973 upper=2.8973 effort=87 velocity=2.1750

File: assets/inspire_hand/inspire_hand_left.urdf (robot description, URDF)
Before this commit: robot h1, 18 links, 17 joints
Joints:
- joint L_index_proximal_joint: limit lower=0 upper=1.3090 effort=1 velocity=0.5 -> lower=0.3377 upper=1.6467 effort=1 velocity=0.5
- joint L_middle_proximal_joint: limit lower=0 upper=1.3090 effort=1 velocity=0.5 -> lower=0.3377 upper=1.6467 effort=1 velocity=0.5
- joint L_pinky_proximal_joint: limit lower=0 upper=1.3090 effort=1 velocity=0.5 -> lower=0.3377 upper=1.6467 effort=1 velocity=0.5
- joint L_ring_proximal_joint: limit lower=0 upper=1.3090 effort=1 velocity=0.5 -> lower=0.3377 upper=1.6467 effort=1 velocity=0.5
- joint L_thumb_distal_joint: mimic joint=L_thumb_proximal_pitch_joint multiplier=0.864 offset=0.907 -> joint=L_thumb_proximal_pitch_joint multiplier=0.667 offset=0
- joint L_thumb_intermediate_joint: mimic joint=L_thumb_proximal_pitch_joint multiplier=1.142 offset=0.490 -> joint=L_thumb_proximal_pitch_joint multiplier=1.334 offset=0
- joint L_thumb_proximal_yaw_joint: limit lower=0.0 upper=1.3090 effort=1 velocity=0.5 -> lower=0.3367 upper=1.4990 effort=1 velocity=0.5

File: assets/inspire_hand/inspire_hand_right.urdf (robot description, URDF)
Before this commit: robot h1, 18 links, 17 joints
Joints:
- joint R_index_proximal_joint: limit lower=0 upper=1.3090 effort=1 velocity=0.5 -> lower=0.3377 upper=1.6467 effort=1 velocity=0.5
- joint R_middle_proximal_joint: limit lower=0 upper=1.3090 effort=1 velocity=0.5 -> lower=0.3377 upper=1.6467 effort=1 velocity=0.5
- joint R_pinky_proximal_joint: limit lower=0 upper=1.3090 effort=1 velocity=0.5 -> lower=0.3377 upper=1.6467 effort=1 velocity=0.5
- joint R_ring_proximal_joint: limit lower=0 upper=1.3090 effort=1 velocity=0.5 -> lower=0.3377 upper=1.6467 effort=1 velocity=0.5
- joint R_thumb_proximal_yaw_joint: limit lower=0 upper=1.3090 effort=1 velocity=0.5 -> lower=0.3367 upper=1.4990 effort=1 velocity=0.5
