Commit message: Rewrite code and update new functions

File: assets/franka_inspire_hand/franka_description/robots/franka_panda_left.urdf (robot description, URDF)
Before this commit: robot panda, 26 links, 25 joints
Links:
- removed link L_hand_base_link
- removed link L_index_intermediate
- removed link L_index_proximal
- removed link L_index_tip
- removed link L_middle_intermediate
- removed link L_middle_proximal
- removed link L_middle_tip
- removed link L_pinky_intermediate
- removed link L_pinky_proximal
- removed link L_pinky_tip
- removed link L_ring_intermediate
- removed link L_ring_proximal
- removed link L_ring_tip
- removed link L_thumb_distal
- removed link L_thumb_intermediate
- removed link L_thumb_proximal
- removed link L_thumb_proximal_base
- removed link L_thumb_tip
- added link hand_base_link, mass 0.14143; collision box size=0.0125 0.0111 0.0089; collision box size=0.0125 0.0111 0.0089
- added link index_intermediate, mass 0.0045683; collision mesh filename=meshes/collision/left_index_intermediate.obj; visual mesh filename=meshes/visual/left_index_intermediate.glb
- added link index_proximal, mass 0.0042403; collision mesh filename=meshes/collision/left_index_proximal.obj; visual mesh filename=meshes/visual/left_index_proximal.glb
- added link index_tip
- added link middle_intermediate, mass 0.0050396; collision mesh filename=meshes/collision/left_middle_intermediate.obj; visual mesh filename=meshes/visual/left_middle_intermediate.glb
- added link middle_proximal, mass 0.0042403; collision mesh filename=meshes/collision/left_index_proximal.obj; visual mesh filename=meshes/visual/left_index_proximal.glb
- added link middle_tip
- added link pinky_intermediate, mass 0.0035996; collision mesh filename=meshes/collision/left_pinky_intermediate.obj; visual mesh filename=meshes/visual/left_pinky_intermediate.glb
- added link pinky_proximal, mass 0.0042403; collision mesh filename=meshes/collision/left_index_proximal.obj; visual mesh filename=meshes/visual/left_index_proximal.glb
- added link pinky_tip
- added link ring_intermediate, mass 0.0045683; collision mesh filename=meshes/collision/left_index_intermediate.obj; visual mesh filename=meshes/visual/left_index_intermediate.glb
- added link ring_proximal, mass 0.0042403; collision mesh filename=meshes/collision/left_index_proximal.obj; visual mesh filename=meshes/visual/left_index_proximal.glb
- added link ring_tip
- added link thumb_distal, mass 0.0033441; collision mesh filename=meshes/collision/left_thumb_distal.obj scale=1 1 1; visual mesh filename=meshes/visual/left_thumb_distal.glb
- added link thumb_intermediate, mass 0.0037847; collision mesh filename=meshes/collision/left_thumb_intermediate.obj; visual mesh filename=meshes/visual/left_thumb_intermediate.glb
- added link thumb_proximal, mass 0.0066075; collision mesh filename=meshes/collision/left_thumb_proximal.obj; visual mesh filename=meshes/visual/left_thumb_proximal.glb
- added link thumb_proximal_base, mass 0.0018869; collision mesh filename=meshes/collision/left_thumb_proximal_base.obj; visual mesh filename=meshes/visual/left_thumb_proximal_base.glb
- added link thumb_tip
- added link wrist_connnect; collision mesh filename=package://franka_description/meshes/collision/wrist_connect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; visual mesh filename=package://franka_description/meshes/visual/wrist_connect5.S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
Joints:
- removed joint L_index_intermediate_joint
- removed joint L_index_proximal_joint
- removed joint L_index_tip_joint
- removed joint L_middle_intermediate_joint
- removed joint L_middle_proximal_joint
- removed joint L_middle_tip_joint
- removed joint L_pinky_intermediate_joint
- removed joint L_pinky_proximal_joint
- removed joint L_pinky_tip_joint
- removed joint L_ring_intermediate_joint
- removed joint L_ring_proximal_joint
- removed joint L_ring_tip_joint
- removed joint L_thumb_distal_joint
- removed joint L_thumb_intermediate_joint
- removed joint L_thumb_proximal_pitch_joint
- removed joint L_thumb_proximal_yaw_joint
- removed joint L_thumb_tip_joint
- removed joint panda_hand_joint
- added joint arm_wrist_joint: type fixed, parent panda_link7, child wrist_connnect, origin xyz=0 0 0.116 rpy=-1.5707963 0 -1.5707963267948966
- added joint index_intermediate_joint: type revolute, parent index_proximal, child index_intermediate, origin xyz=-0.0026138 -0.032026 -0.001 rpy=0 0 0, axis 0 0 -1, limit lower=-0.04545 upper=1.56 effort=1 velocity=0.5, mimic joint=index_proximal_joint multiplier=1.06399 offset=-0.04545
- added joint index_proximal_joint: type revolute, parent hand_base_link, child index_proximal, origin xyz=0.00028533 -0.13653 0.032268 rpy=-0.034907 0 0, axis 0 0 -1, limit lower=0 upper=1.47 effort=1 velocity=0.5
- added joint index_tip_joint: type fixed, parent index_intermediate, child index_tip, origin xyz=-0.0008 -0.045 -0.005 rpy=0 0 0
- added joint middle_intermediate_joint: type revolute, parent middle_proximal, child middle_intermediate, origin xyz=-0.0024229 -0.032041 -0.001 rpy=0 0 0, axis 0 0 -1, limit lower=-0.04545 upper=1.56 effort=1 velocity=0.5, mimic joint=middle_proximal_joint multiplier=1.06399 offset=-0.04545
- added joint middle_proximal_joint: type revolute, parent hand_base_link, child middle_proximal, origin xyz=0.00028533 -0.1371 0.01295 rpy=0 0 0, axis 0 0 -1, limit lower=0 upper=1.47 effort=1 velocity=0.5
- added joint middle_tip_joint: type fixed, parent middle_intermediate, child middle_tip, origin xyz=-0.001 -0.048 -0.005 rpy=0 0 0
- added joint pinky_intermediate_joint: type revolute, parent pinky_proximal, child pinky_intermediate, origin xyz=-0.0024229 -0.032041 -0.001 rpy=0 0 0, axis 0 0 -1, limit lower=-0.04545 upper=1.56 effort=1 velocity=0.5, mimic joint=pinky_proximal_joint multiplier=1.06399 offset=-0.04545
- added joint pinky_proximal_joint: type revolute, parent hand_base_link, child pinky_proximal, origin xyz=0.00028533 -0.13571 -0.025488 rpy=0.10472 0 0, axis 0 0 -1, limit lower=0 upper=1.47 effort=1 velocity=0.5
- added joint pinky_tip_joint: type fixed, parent pinky_intermediate, child pinky_tip, origin xyz=-0.0008 -0.037 -0.005 rpy=0 0 0
- added joint ring_intermediate_joint: type revolute, parent ring_proximal, child ring_intermediate, origin xyz=-0.0024229 -0.032041 -0.001 rpy=0 0 0, axis 0 0 -1, limit lower=-0.04545 upper=1.56 effort=1 velocity=0.5, mimic joint=ring_proximal_joint multiplier=1.06399 offset=-0.04545
- added joint ring_proximal_joint: type revolute, parent hand_base_link, child ring_proximal, origin xyz=0.00028533 -0.13691 -0.0062872 rpy=0.05236 0 0, axis 0 0 -1, limit lower=0 upper=1.47 effort=1 velocity=0.5
- added joint ring_tip_joint: type fixed, parent ring_intermediate, child ring_tip, origin xyz=-0.0008 -0.045 -0.005 rpy=0 0 0
- added joint thumb_distal_joint: type revolute, parent thumb_intermediate, child thumb_distal, origin xyz=0.020248 -0.010156 -0.0012 rpy=0 0 0, axis 0 0 -1, limit lower=0 upper=0.4 effort=1 velocity=0.5, mimic joint=thumb_proximal_pitch_joint multiplier=0.667 offset=0
- added joint thumb_intermediate_joint: type revolute, parent thumb_proximal, child thumb_intermediate, origin xyz=0.04407 -0.034553 -0.0008 rpy=0 0 0, axis 0 0 -1, limit lower=0 upper=0.8 effort=1 velocity=0.5, mimic joint=thumb_proximal_pitch_joint multiplier=1.334 offset=0
- added joint thumb_proximal_pitch_joint: type revolute, parent thumb_proximal_base, child thumb_proximal, origin xyz=0.0099867 0.0098242 -0.0089 rpy=-1.5708 0 0.16939, axis 0 0 -1, limit lower=0 upper=0.6 effort=1 velocity=0.5
- added joint thumb_proximal_yaw_joint: type revolute, parent hand_base_link, child thumb_proximal_base, origin xyz=-0.01696 -0.0691 0.02045 rpy=1.5708 -1.5708 0, axis 0 0 1, limit lower=0 upper=1.308 effort=1 velocity=0.5
- added joint thumb_tip_joint: type fixed, parent thumb_distal, child thumb_tip, origin xyz=0.0202 -0.0140 -0.006 rpy=0 0 0
- added joint wrist_hand_joint: type fixed, parent wrist_connnect, child hand_base_link, origin xyz=0 -0.02696 0.0447 rpy=-1.5707963 0 1.5707963267948966
- joint panda_joint1: limit lower=-2.8973 upper=2.8973 effort=87 velocity=2.1750 -> lower=-2.7437 upper=2.7437 effort=87 velocity=2.62
- joint panda_joint2: limit lower=-1.7628 upper=1.7628 effort=87 velocity=2.1750 -> lower=-1.7837 upper=1.7837 effort=87 velocity=2.62
- joint panda_joint3: limit lower=-2.8973 upper=2.8973 effort=87 velocity=2.1750 -> lower=-2.9007 upper=2.9007 effort=87 velocity=2.62
- joint panda_joint4: limit lower=-3.0718 upper=-0.0698 effort=87 velocity=2.1750 -> lower=-3.0421 upper=-0.1518 effort=87 velocity=2.62
- joint panda_joint5: limit lower=-2.8973 upper=2.8973 effort=12 velocity=2.6100 -> lower=-2.8065 upper=2.8065 effort=12 velocity=5.26
- joint panda_joint6: limit lower=-0.0175 upper=3.7525 effort=12 velocity=2.6100 -> lower=0.5445 upper=4.5169 effort=12 velocity=4.18
- joint panda_joint7: limit lower=-2.8973 upper=2.8973 effort=12 velocity=2.6100 -> lower=-3.0159 upper=3.0159 effort=12 velocity=5.26

File: assets/franka_inspire_hand/franka_description/robots/franka_panda_right.urdf (robot description, URDF)
Before this commit: robot panda, 26 links, 25 joints
Links:
- added link wrist_connnect; collision mesh filename=package://franka_description/meshes/collision/wrist_connect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; visual mesh filename=package://franka_description/meshes/visual/wrist_connect5.S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
Joints:
- removed joint panda_hand_joint
- added joint arm_wrist_joint: type fixed, parent panda_link7, child wrist_connnect, origin xyz=0 0 0.116 rpy=-1.5707963 0 -1.5707963267948966
- added joint wrist_hand_joint: type fixed, parent wrist_connnect, child hand_base_link, origin xyz=0 -0.02696 0.0447 rpy=-1.5707963 0 1.5707963267948966
- joint panda_joint1: limit lower=-2.8973 upper=2.8973 effort=87 velocity=2.1750 -> lower=-2.7437 upper=2.7437 effort=87 velocity=2.62
- joint panda_joint2: limit lower=-1.7628 upper=1.7628 effort=87 velocity=2.1750 -> lower=-1.7837 upper=1.7837 effort=87 velocity=2.62
- joint panda_joint3: limit lower=-2.8973 upper=2.8973 effort=87 velocity=2.1750 -> lower=-2.9007 upper=2.9007 effort=87 velocity=2.62
- joint panda_joint4: limit lower=-3.0718 upper=-0.0698 effort=87 velocity=2.1750 -> lower=-3.0421 upper=-0.1518 effort=87 velocity=2.62
- joint panda_joint5: limit lower=-2.8973 upper=2.8973 effort=12 velocity=2.6100 -> lower=-2.8065 upper=2.8065 effort=12 velocity=5.26
- joint panda_joint6: limit lower=-0.0175 upper=3.7525 effort=12 velocity=2.6100 -> lower=0.5445 upper=4.5169 effort=12 velocity=4.18
- joint panda_joint7: limit lower=-2.8973 upper=2.8973 effort=12 velocity=2.6100 -> lower=-3.0159 upper=3.0159 effort=12 velocity=5.26

File: assets/franka_pinocchio/robots/franka_panda.urdf (robot description, URDF)
Before this commit: robot panda, 8 links, 7 joints
Links:
- added link hand_base_link, mass 0.14143; collision box size=0.0125 0.0111 0.0089; collision box size=0.0125 0.0111 0.0089
- added link wrist_connnect; collision mesh filename=file:///home/zhourui/Desktop/user/project/dex-mimic/assets/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; visual mesh filename=file:///home/zhourui/Desktop/user/project/dex-mimic/assets/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
Joints:
- added joint arm_wrist_joint: type fixed, parent panda_link7, child wrist_connnect, origin xyz=0 0 0.116 rpy=-1.5707963 0 -1.5707963267948966
- added joint wrist_hand_joint: type fixed, parent wrist_connnect, child hand_base_link, origin xyz=0 -0.02696 0.0447 rpy=-1.5707963 0 1.5707963267948966

File: assets/inspire_hand/inspire_hand_left.urdf (robot description, URDF)
Before this commit: robot h1, 18 links, 17 joints
Joints:
- joint L_index_intermediate_joint: mimic joint=L_index_proximal_joint multiplier=1.117 offset=-0.187 -> joint=L_index_proximal_joint multiplier=1 offset=0
- joint L_index_proximal_joint: limit lower=0.3377 upper=1.6467 effort=1 velocity=0.5 -> lower=0 upper=1.7 effort=1 velocity=0.5
- joint L_middle_intermediate_joint: mimic joint=L_middle_proximal_joint multiplier=1.117 offset=-0.187 -> joint=L_middle_proximal_joint multiplier=1 offset=0
- joint L_middle_proximal_joint: limit lower=0.3377 upper=1.6467 effort=1 velocity=0.5 -> lower=0 upper=1.7 effort=1 velocity=0.5
- joint L_pinky_intermediate_joint: mimic joint=L_pinky_proximal_joint multiplier=1.117 offset=-0.187 -> joint=L_pinky_proximal_joint multiplier=1 offset=0
- joint L_pinky_proximal_joint: limit lower=0.3377 upper=1.6467 effort=1 velocity=0.5 -> lower=0 upper=1.7 effort=1 velocity=0.5
- joint L_ring_intermediate_joint: mimic joint=L_ring_proximal_joint multiplier=1.117 offset=-0.187 -> joint=L_ring_proximal_joint multiplier=1 offset=0
- joint L_ring_proximal_joint: limit lower=0.3377 upper=1.6467 effort=1 velocity=0.5 -> lower=0 upper=1.7 effort=1 velocity=0.5
- joint L_thumb_distal_joint: mimic joint=L_thumb_proximal_pitch_joint multiplier=0.667 offset=0 -> joint=L_thumb_proximal_pitch_joint multiplier=2.4 offset=0
- joint L_thumb_intermediate_joint: mimic joint=L_thumb_proximal_pitch_joint multiplier=1.334 offset=0 -> joint=L_thumb_proximal_pitch_joint multiplier=1.6 offset=0
- joint L_thumb_proximal_pitch_joint: limit lower=0.0 upper=0.4712 effort=1 velocity=0.5 -> lower=0.0 upper=0.5 effort=1 velocity=0.5
- joint L_thumb_proximal_yaw_joint: limit lower=0.3367 upper=1.4990 effort=1 velocity=0.5 -> lower=-0.1 upper=1.3 effort=1 velocity=0.5

File: assets/inspire_hand/inspire_hand_right.urdf (robot description, URDF)
Before this commit: robot h1, 18 links, 17 joints
Joints:
- joint R_index_proximal_joint: limit lower=0.3377 upper=1.6467 effort=1 velocity=0.5 -> lower=0 upper=1.7 effort=1 velocity=0.5
- joint R_middle_intermediate_joint: mimic joint=R_middle_proximal_joint multiplier=1.117 offset=-0.187 -> joint=R_middle_proximal_joint multiplier=1 offset=0
- joint R_middle_proximal_joint: limit lower=0.3377 upper=1.6467 effort=1 velocity=0.5 -> lower=0 upper=1.7 effort=1 velocity=0.5
- joint R_pinky_intermediate_joint: mimic joint=R_pinky_proximal_joint multiplier=1.117 offset=-0.187 -> joint=R_pinky_proximal_joint multiplier=1 offset=0
- joint R_pinky_proximal_joint: limit lower=0.3377 upper=1.6467 effort=1 velocity=0.5 -> lower=0 upper=1.7 effort=1 velocity=0.5
- joint R_ring_intermediate_joint: mimic joint=R_ring_proximal_joint multiplier=1.117 offset=-0.187 -> joint=R_ring_proximal_joint multiplier=1 offset=0
- joint R_ring_proximal_joint: limit lower=0.3377 upper=1.6467 effort=1 velocity=0.5 -> lower=0 upper=1.7 effort=1 velocity=0.5
- joint R_thumb_distal_joint: mimic joint=R_thumb_proximal_pitch_joint multiplier=0.864 offset=0.907 -> joint=R_thumb_proximal_pitch_joint multiplier=2.4 offset=0
- joint R_thumb_intermediate_joint: mimic joint=R_thumb_proximal_pitch_joint multiplier=1.142 offset=0.490 -> joint=R_thumb_proximal_pitch_joint multiplier=1.6 offset=0
- joint R_thumb_proximal_pitch_joint: limit lower=0.0 upper=0.4712 effort=1 velocity=0.5 -> lower=0.0 upper=0.5 effort=1 velocity=0.5
- joint R_thumb_proximal_yaw_joint: limit lower=0.3367 upper=1.4990 effort=1 velocity=0.5 -> lower=-0.1 upper=1.3 effort=1 velocity=0.5
