Commit message: Fix package path bug in URDF

File: assets/franka_pinocchio/robots/franka_panda.urdf (robot description, URDF)
Before this commit: robot panda, 10 links, 9 joints
Links:
- link hand_base_link: geometry collision box size=0.0125 0.0111 0.0089; collision box size=0.0125 0.0111 0.0089
- link panda_link0: geometry collision mesh filename=package://franka_pinocchio/meshes/collision/link0.obj; visual mesh filename=package://franka_pinocchio/meshes/visual/link0.dae
- link panda_link1: geometry collision mesh filename=package://franka_pinocchio/meshes/collision/link1.obj; visual mesh filename=package://franka_pinocchio/meshes/visual/link1.dae
- link panda_link2: geometry collision mesh filename=package://franka_pinocchio/meshes/collision/link2.obj; visual mesh filename=package://franka_pinocchio/meshes/visual/link2.dae
- link panda_link3: geometry collision mesh filename=package://franka_pinocchio/meshes/collision/link3.obj; visual mesh filename=package://franka_pinocchio/meshes/visual/link3.dae
- link panda_link4: geometry collision mesh filename=package://franka_pinocchio/meshes/collision/link4.obj; visual mesh filename=package://franka_pinocchio/meshes/visual/link4.dae
- link panda_link5: geometry collision mesh filename=package://franka_pinocchio/meshes/collision/link5.obj; visual mesh filename=package://franka_pinocchio/meshes/visual/link5.dae
- link panda_link6: geometry collision mesh filename=package://franka_pinocchio/meshes/collision/link6.obj; visual mesh filename=package://franka_pinocchio/meshes/visual/link6.dae
- link panda_link7: geometry collision mesh filename=package://franka_pinocchio/meshes/collision/link7.obj; visual mesh filename=package://franka_pinocchio/meshes/visual/link7.dae
- link wrist_connnect: geometry collision mesh filename=package://franka_pinocchio/meshes/visual/wrist_connect5.STL; visual mesh filename=package://franka_pinocchio/meshes/visual/wrist_connect5.STL
